File: firmware/TP1/TP1.kicad_sch (KiCad schematic)
At the start: 27 parts, among them J1 Conn_02x07_Odd_Even, J2 INPUT, J3 POWER, J4 OUTPUT, U1 BU33SD5WG-TR, U2 STM32L021K4Tx, U3 MCP4801

Commit message: kicad
Connections:
- net  USART2_TX is gone; now on net USART2_TX: U2.8 (PA2)
- net ADC_ IN1 is gone; now on net ADC_IN1: U2.7 (PA1)
- net SYS_SWDCLK is gone; now on net SWDCK: U2.24 (PA14)
- net SYS_SWDIO is gone; now on net SWDIO: U2.23 (PA13)
- net TIM2_CH1 is gone; now on net LED_STATUS: U2.18 (PA8)
- net +3.3V: no longer C5.1, C6.1, L1.2
- net +3.3VA: now also C5.1, C6.1, L1.2
- net SPI1_MISO: no longer names the net of U2.12 (PA6)
- no-connect marks 19 -> 20
Other:
- note added: "MISO NOT CONNECTED"
Changed lines of the file:
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@@
   (no_connect (at 81.28 97.79))
   (no_connect (at 106.68 92.71))
+  (no_connect (at 113.03 82.55))
   (no_connect (at 55.88 160.02))
   (no_connect (at 106.68 97.79))
@@
     (effects (font (size 1.27 1.27)) (justify right bottom))
   )
+  (text "MISO NOT CONNECTED\n" (at 114.3 83.82 0)
+    (effects (font (size 1.27 1.27)) (justify left bottom))
+  )
   (text "IO Connectors" (at 77.47 139.7 0)
     (effects (font (size 1.27 1.27)) (justify left bottom))
@@
     )
   )
-  (global_label "SYS_SWDCLK" (shape input) (at 113.03 102.87 0) (fields_autoplaced)
-    (effects (font (size 1 1)) (justify left))
-    (property "Intersheet References" "${INTERSHEET_REFS}" (id 0) (at 124.3586 102.8075 0)
+  (global_label "SWDCK" (shape input) (at 113.03 102.87 0) (fields_autoplaced)
+    (effects (font (size 1 1)) (justify left))
+    (property "Intersheet References" "${INTERSHEET_REFS}" (id 0) (at 120.0252 102.8075 0)
       (effects (font (size 1 1)) (justify left) hide)
     )
@@
     )
   )
-  (global_label " USART2_TX" (shape input) (at 113.03 72.39 0) (fields_autoplaced)
-    (effects (font (size 1 1)) (justify left))
-    (property "Intersheet References" "${INTERSHEET_REFS}" (id 0) (at 123.7395 72.3275 0)
+  (global_label "USART2_TX" (shape input) (at 113.03 72.39 0) (fields_autoplaced)
+    (effects (font (size 1 1)) (justify left))
+    (property "Intersheet References" "${INTERSHEET_REFS}" (id 0) (at 122.9776 72.3275 0)
       (effects (font (size 1 1)) (justify left) hide)
     )
@@
     (effects (font (size 1 1)) (justify left))
     (property "Intersheet References" "${INTERSHEET_REFS}" (id 0) (at 61.5419 165.0375 0)
-      (effects (font (size 1 1)) (justify left) hide)
-    )
-  )
-  (global_label "SPI1_MISO" (shape input) (at 113.03 82.55 0) (fields_autoplaced)
-    (effects (font (size 1 1)) (justify left))
-    (property "Intersheet References" "${INTERSHEET_REFS}" (id 0) (at 122.6919 82.4875 0)
       (effects (font (size 1 1)) (justify left) hide)
     )
@@
     )
   )
-  (global_label "TIM2_CH1" (shape input) (at 113.03 87.63 0) (fields_autoplaced)
-    (effects (font (size 1 1)) (justify left))
-    (property "Intersheet References" "${INTERSHEET_REFS}" (id 0) (at 122.0252 87.5675 0)
+  (global_label "LED_STATUS" (shape input) (at 113.03 87.63 0) (fields_autoplaced)
+    (effects (font (size 1 1)) (justify left))
+    (property "Intersheet References" "${INTERSHEET_REFS}" (id 0) (at 123.7395 87.5675 0)
       (effects (font (size 1 1)) (justify left) hide)
     )
@@
     )
   )
-  (global_label "ADC_ IN1" (shape input) (at 113.03 69.85 0) (fields_autoplaced)
-    (effects (font (size 1 1)) (justify left))
-    (property "Intersheet References" "${INTERSHEET_REFS}" (id 0) (at 121.7871 69.7875 0)
+  (global_label "ADC_IN1" (shape input) (at 113.03 69.85 0) (fields_autoplaced)
+    (effects (font (size 1 1)) (justify left))
+    (property "Intersheet References" "${INTERSHEET_REFS}" (id 0) (at 121.0252 69.7875 0)
       (effects (font (size 1 1)) (justify left) hide)
     )
@@
     )
   )
-  (global_label "SYS_SWDIO" (shape input) (at 113.03 100.33 0) (fields_autoplaced)
-    (effects (font (size 1 1)) (justify left))
-    (property "Intersheet References" "${INTERSHEET_REFS}" (id 0) (at 123.0729 100.2675 0)
+  (global_label "SWDIO" (shape input) (at 113.03 100.33 0) (fields_autoplaced)
+    (effects (font (size 1 1)) (justify left))
+    (property "Intersheet References" "${INTERSHEET_REFS}" (id 0) (at 119.549 100.2675 0)
       (effects (font (size 1 1)) (justify left) hide)
     )
@@
     (pin "1")
   )
+  (symbol (lib_id "power:+3.3VA") (at 133.35 29.21 0) (unit 1)
+    (in_bom yes) (on_board yes) (fields_autoplaced)
+    (property "Reference" "#PWR0102" (id 0) (at 133.35 33.02 0)
+      (effects (font (size 1.27 1.27)) hide)
+    )
+    (property "Value" "+3.3VA" (id 1) (at 133.35 24.13 0))
+    (property "Footprint" "" (id 2) (at 133.35 29.21 0)
+      (effects (font (size 1.27 1.27)) hide)
+    )
+    (property "Datasheet" "" (id 3) (at 133.35 29.21 0)
+      (effects (font (size 1.27 1.27)) hide)
+    )
+    (pin "1")
+  )
   (symbol (lib_id "Device:LED") (at 261.62 111.76 90) (unit 1)
     (in_bom yes) (on_board yes) (fields_autoplaced)
@@
     (pin "1")
     (pin "2")
-  )
-  (symbol (lib_id "power:+3.3V") (at 133.35 29.21 0) (unit 1)
-    (in_bom yes) (on_board yes) (fields_autoplaced)
-    (property "Reference" "#PWR016" (id 0) (at 133.35 33.02 0)
-      (effects (font (size 1.27 1.27)) hide)
-    )
-    (property "Value" "+3.3V" (id 1) (at 133.35 24.13 0))
-    (property "Footprint" "" (id 2) (at 133.35 29.21 0)
-      (effects (font (size 1.27 1.27)) hide)
-    )
-    (property "Datasheet" "" (id 3) (at 133.35 29.21 0)
-      (effects (font (size 1.27 1.27)) hide)
-    )
-    (pin "1")
   )
   (symbol (lib_id "Device:R") (at 261.62 121.92 0) (unit 1)
@@
       (reference "#PWR015") (unit 1) (value "GND") (footprint "")
     )
-    (path "/a3d8624e-2bf8-48b0-b5b9-2bc4456397e3"
-      (reference "#PWR016") (unit 1) (value "+3.3V") (footprint "")
-    )
     (path "/8eeeab67-739f-473b-9b3f-4c84ec7950ba"
       (reference "#PWR017") (unit 1) (value "+5V") (footprint "")
@@
       (reference "#PWR0101") (unit 1) (value "GND") (footprint "")
     )
+    (path "/2ff1bc67-dfc9-48be-b239-aa8e7fa8cb90"
+      (reference "#PWR0102") (unit 1) (value "+3.3VA") (footprint "")
+    )
     (path "/5c8866b6-3678-4775-b51e-b8276b448a1e"
